File: Proyecto_1.kicad_sch (KiCad schematic)
At the start: 2 parts

Commit message: ahora Proyecto_1.kicad_sch tiene un nuevo resistor
Parts:
- added R?: R, Resistor_THT:R_Axial_DIN0204_L3.6mm_D1.6mm_P7.62mm_Horizontal, symbol Device:R
Connections:
- net +5V: now also R?.2
- net at D1.2 (A), R1.1: now also R?.1
Changed lines of the file:
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@@
   (junction (at 161.29 90.17) (diameter 0) (color 0 0 0 0)
+  )
+  (junction (at 148.59 90.17) (diameter 0) (color 0 0 0 0)
   )
   (junction (at 137.16 90.17) (diameter 0) (color 0 0 0 0)
   )
+  (wire (pts (xy 148.59 80.518) (xy 148.59 90.17))
+    (stroke (width 0) (type default) (color 0 0 0 0))
+  )
   (wire (pts (xy 138.43 90.17) (xy 137.16 90.17))
+    (stroke (width 0) (type default) (color 0 0 0 0))
+  )
+  (wire (pts (xy 159.258 80.518) (xy 161.544 80.772))
+    (stroke (width 0) (type default) (color 0 0 0 0))
+  )
+  (wire (pts (xy 148.59 90.17) (xy 151.13 90.17))
     (stroke (width 0) (type default) (color 0 0 0 0))
   )
@@
   )
   (wire (pts (xy 162.56 90.17) (xy 161.29 90.17))
+    (stroke (width 0) (type default) (color 0 0 0 0))
+  )
+  (wire (pts (xy 161.544 80.772) (xy 161.29 90.17))
     (stroke (width 0) (type default) (color 0 0 0 0))
   )
@@
     (stroke (width 0) (type default) (color 0 0 0 0))
   )
+  (wire (pts (xy 151.384 80.518) (xy 148.59 80.518))
+    (stroke (width 0) (type default) (color 0 0 0 0))
+  )
   (polyline (pts (xy 129.54 76.2) (xy 168.91 76.2))
     (stroke (width 0) (type default) (color 0 0 0 0))
@@
     (stroke (width 0) (type default) (color 0 0 0 0))
   )
-  (wire (pts (xy 146.05 90.17) (xy 151.13 90.17))
+  (wire (pts (xy 146.05 90.17) (xy 148.59 90.17))
     (stroke (width 0) (type default) (color 0 0 0 0))
   )
@@
   )
   (wire (pts (xy 162.56 86.36) (xy 162.56 90.17))
+    (stroke (width 0) (type default) (color 0 0 0 0))
+  )
+  (wire (pts (xy 159.258 80.518) (xy 159.004 80.518))
     (stroke (width 0) (type default) (color 0 0 0 0))
   )
@@
   (text "Current\nlimiting \nresistor" (at 152.4 97.79 0)
     (effects (font (size 1.27 1.27)) (justify left bottom))
+  )
+  (symbol (lib_id "Device:R") (at 155.194 80.518 90) (unit 1)
+    (in_bom yes) (on_board yes) (fields_autoplaced)
+    (property "Reference" "R?" (id 0) (at 155.194 74.168 90))
+    (property "Value" "R" (id 1) (at 155.194 76.708 90))
+    (property "Footprint" "Resistor_THT:R_Axial_DIN0204_L3.6mm_D1.6mm_P7.62mm_Horizontal" (id 2) (at 155.194 82.296 90)
+      (effects (font (size 1.27 1.27)) hide)
+    )
+    (property "Datasheet" "~" (id 3) (at 155.194 80.518 0)
+      (effects (font (size 1.27 1.27)) hide)
+    )
+    (pin "1")
+    (pin "2")
   )
   (symbol (lib_id "power:PWR_FLAG") (at 137.16 85.09 0) (unit 1)
@@
       (reference "R1") (unit 1) (value "R") (footprint "Resistor_THT:R_Axial_DIN0204_L3.6mm_D1.6mm_P7.62mm_Horizontal")
     )
+    (path "/0554bea0-89b2-4e25-9ea3-4c73921c94cb"
+      (reference "R?") (unit 1) (value "R") (footprint "Resistor_THT:R_Axial_DIN0204_L3.6mm_D1.6mm_P7.62mm_Horizontal")
+    )
   )
